File: Hardware/Hardware.kicad_sch (KiCad schematic)
At the start: 62 parts, among them J1 USB_C_Receptacle_USB2.0_16P, J2 PICO_PINOUT, Q1 BSS138, Q2 BSS138, U1 AP33772S, U10 TPS62933DRLR, U3 W25Q16JVUXIQ_TR, U4 RP2040, U5 AON7262E, U6 AON7262E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

Commit message: Update BOM
Parts:
- D1, D2: LCSC C72043 -> C12624
- Q2: JLCPCB Rotation Offset (none) -> 180
Changed lines of the file:
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@@
 			)
 		)
+		(property "JLCPCB Rotation Offset" "180"
+			(at 111.76 124.46 90)
+			(effects
+				(font
+					(size 1.27 1.27)
+				)
+				(hide yes)
+			)
+		)
 		(pin "1"
 		)
@@
 			)
 		)
-		(property "LCSC" "C72043"
+		(property "LCSC" "C12624"
 			(at 207.645 181.61 90)
 			(effects
@@
 			)
 		)
-		(property "LCSC" "C72043"
+		(property "LCSC" "C12624"
 			(at 160.02 190.5 90)
 			(effects
